File: lap-counter/_autosave-lap-counter.kicad_sch (KiCad schematic)
At the start: 23 parts, among them U1 TLP3543

Commit message: Review and raise version to v1.0
Parts:
- renumbered A1 to AR1
Changed lines of the file:
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@@
   (symbol (lib_id "MCU_Module:Arduino_Nano_v3.x") (at 101.6 106.68 180) (unit 1)
     (in_bom yes) (on_board yes) (fields_autoplaced)
-    (property "Reference" "A1" (id 0) (at 104.3687 78.74 0)
+    (property "Reference" "AR1" (id 0) (at 104.3687 78.74 0)
       (effects (font (size 1.27 1.27)) (justify right))
     )
@@
     )
     (path "/925356e8-9fe3-4fca-8329-eba967a76629"
-      (reference "A1") (unit 1) (value "Arduino_Nano_v3.x") (footprint "Module:Arduino_Nano")
+      (reference "AR1") (unit 1) (value "Arduino_Nano_v3.x") (footprint "Module:Arduino_Nano")
     )
     (path "/ca4eb5d8-f726-41a3-999b-d20db9f92b52"
